Commit message: Simulation/ros2: update URDF to display J1 parts
Update URDF MCU base and J1 links.
The joint element describes the kinematics and dynamics of the joint.
The current origin element in joint is derived from FreeCAD assembly
workbench where it list detail about the desired xyz.

Signed-off-by: KizEvo <vandungqc03@gmail.com>

File: Simulation/ros2/src/arm_desc/buddyarm_urdf/src/robot_arm.urdf.xacro (robot description, xacro)
@@ -1,10 +1,73 @@
 <?xml version="1.0"?>
 <robot xmlns:xacro="http://www.ros.org/wiki/xacro" name="BuddyArm">
-  <link name="base_link">
+  <!--
+  =============================================================
+                              LINKS
+  Origin values based on FreeCAD assembly translation and
+  rotation
+  =============================================================
+   -->
+  <link name="mcu_base_link">
     <visual>
       <geometry>
-        <cylinder length="0.6" radius="0.2"/>
+        <mesh filename="package://buddyarm_urdf/mesh/buddy_arm-Base.dae"/>
       </geometry>
     </visual>
   </link>
+  <link name="j1_base_link">
+    <visual>
+      <geometry>
+        <mesh filename="package://buddyarm_urdf/mesh/buddy_arm-J1_Base.dae"/>
+      </geometry>
+    </visual>
+  </link>
+  <link name="j1_turret_housing_link">
+    <visual>
+      <geometry>
+        <mesh filename="package://buddyarm_urdf/mesh/buddy_arm-J1_Turret_Housing.dae"/>
+      </geometry>
+    </visual>
+  </link>
+  <link name="j1_platform_link">
+    <visual>
+      <geometry>
+        <mesh filename="package://buddyarm_urdf/mesh/buddy_arm-J1_Platform.dae"/>
+      </geometry>
+    </visual>
+  </link>
+  <link name="j1_spindle_link">
+    <visual>
+      <geometry>
+        <mesh filename="package://buddyarm_urdf/mesh/buddy_arm-J1_Spindle.dae"/>
+      </geometry>
+    </visual>
+  </link>
+  <!--
+  =============================================================
+                              JOINTs
+  Origin values based on FreeCAD assembly translation and
+  rotation
+  - mcu_base is the origin positon 0,0,0
+  =============================================================
+   -->
+  <joint name="mcu_base_to_j1_base_joint" type="fixed">
+    <parent link="mcu_base_link"/>
+    <child link="j1_base_link"/>
+    <origin xyz="0 0.075 0.018"/>
+  </joint>
+  <joint name="mcu_base_to_j1_turret_housing_joint" type="fixed">
+    <parent link="mcu_base_link"/>
+    <child link="j1_turret_housing_link"/>
+    <origin xyz="0 0.225 0.025"/>
+  </joint>
+  <joint name="mcu_base_to_j1_spindle_joint" type="fixed">
+    <parent link="mcu_base_link"/>
+    <child link="j1_spindle_link"/>
+    <origin xyz="0 0.225 -0.007"/>
+  </joint>
+  <joint name="mcu_base_to_j1_platform_link" type="fixed">
+    <parent link="mcu_base_link"/>
+    <child link="j1_platform_link"/>
+    <origin xyz="0 0.225 0.090"/>
+  </joint>
 </robot>

Commit message: Simulation/ros2: add J2 parts in URDF
Signed-off-by: KizEvo <vandungqc03@gmail.com>

File: Simulation/ros2/src/arm_desc/buddyarm_urdf/src/robot_arm.urdf.xacro (robot description, xacro)
@@ -43,4 +43,32 @@
     </visual>
   </link>
+  <link name="j2_arm_link">
+    <visual>
+      <geometry>
+        <mesh filename="package://buddyarm_urdf/mesh/buddy_arm-J2_Arm.dae"/>
+      </geometry>
+    </visual>
+  </link>
+  <link name="j2_spindle_link">
+    <visual>
+      <geometry>
+        <mesh filename="package://buddyarm_urdf/mesh/buddy_arm-J2_Spindle.dae"/>
+      </geometry>
+    </visual>
+  </link>
+  <link name="j2_tension_ring_link">
+    <visual>
+      <geometry>
+        <mesh filename="package://buddyarm_urdf/mesh/buddy_arm-J2_Tension_Ring.dae"/>
+      </geometry>
+    </visual>
+  </link>
+  <link name="j2_turret_housing_link">
+    <visual>
+      <geometry>
+        <mesh filename="package://buddyarm_urdf/mesh/buddy_arm-J2_Turret_Housing.dae"/>
+      </geometry>
+    </visual>
+  </link>
   <!--
   =============================================================
@@ -49,4 +77,6 @@
   rotation
   - mcu_base is the origin positon 0,0,0
+  - see 'Hardware/' under 'phunguyen/basic-assembly' branch,
+   grep for 'zero pose' commit.
   =============================================================
    -->
@@ -66,8 +96,28 @@
     <origin xyz="0 0.225 -0.007"/>
   </joint>
-  <joint name="mcu_base_to_j1_platform_link" type="fixed">
+  <joint name="mcu_base_to_j1_platform_joint" type="fixed">
     <parent link="mcu_base_link"/>
     <child link="j1_platform_link"/>
     <origin xyz="0 0.225 0.090"/>
   </joint>
+  <joint name="mcu_base_to_j2_turret_housing_joint" type="fixed">
+    <parent link="mcu_base_link"/>
+    <child link="j2_turret_housing_link"/>
+    <origin rpy="${pi/2} 0 ${-pi/2}" xyz="-0.021 0.245 0.090"/>
+  </joint>
+  <joint name="mcu_base_to_j2_spindle_joint" type="fixed">
+    <parent link="mcu_base_link"/>
+    <child link="j2_spindle_link"/>
+    <origin rpy="${pi/2} 0 ${pi/2}" xyz="-0.061 0.285 0.140"/>
+  </joint>
+  <joint name="mcu_base_to_j2_tension_ring_joint" type="fixed">
+    <parent link="mcu_base_link"/>
+    <child link="j2_tension_ring_link"/>
+    <origin rpy="${-pi/2} 0 ${pi/2}" xyz="0.010 0.285 0.140"/>
+  </joint>
+  <joint name="mcu_base_to_j2_arm_joint" type="fixed">
+    <parent link="mcu_base_link"/>
+    <child link="j2_arm_link"/>
+    <origin rpy="${pi/2} 0 0" xyz="-0.056 0.315 0.110"/>
+  </joint>
 </robot>

Commit message: Simulation/ros2: add J3 parts in URDF
Signed-off-by: KizEvo <vandungqc03@gmail.com>

File: Simulation/ros2/src/arm_desc/buddyarm_urdf/src/robot_arm.urdf.xacro (robot description, xacro)
@@ -71,4 +71,18 @@
     </visual>
   </link>
+  <link name="j3_bearing_cup_link">
+    <visual>
+      <geometry>
+        <mesh filename="package://buddyarm_urdf/mesh/buddy_arm-J3_Bearing_Cup.dae"/>
+      </geometry>
+    </visual>
+  </link>
+  <link name="j3_spindle_link">
+    <visual>
+      <geometry>
+        <mesh filename="package://buddyarm_urdf/mesh/buddy_arm-J3_Spindle.dae"/>
+      </geometry>
+    </visual>
+  </link>
   <!--
   =============================================================
@@ -121,3 +135,13 @@
     <origin rpy="${pi/2} 0 0" xyz="-0.056 0.315 0.110"/>
   </joint>
+  <joint name="mcu_base_to_j3_bearing_cup_joint" type="fixed">
+    <parent link="mcu_base_link"/>
+    <child link="j3_bearing_cup_link"/>
+    <origin rpy="0 ${-pi/2} 0" xyz="-0.024 0.285 0.373"/>
+  </joint>
+  <joint name="mcu_base_to_j3_spindle_joint" type="fixed">
+    <parent link="mcu_base_link"/>
+    <child link="j3_spindle_link"/>
+    <origin rpy="${pi} ${pi/2} 0" xyz="-0.004 0.285 0.373"/>
+  </joint>
 </robot>

Commit message: Simulation/ros2: add J4 parts in URDF
Signed-off-by: KizEvo <vandungqc03@gmail.com>

File: Simulation/ros2/src/arm_desc/buddyarm_urdf/src/robot_arm.urdf.xacro (robot description, xacro)
@@ -85,4 +85,18 @@
     </visual>
   </link>
+  <link name="j4_turret_housing_link">
+    <visual>
+      <geometry>
+        <mesh filename="package://buddyarm_urdf/mesh/buddy_arm-J4_Turret_Housing.dae"/>
+      </geometry>
+    </visual>
+  </link>
+  <link name="j4_spindle_link">
+    <visual>
+      <geometry>
+        <mesh filename="package://buddyarm_urdf/mesh/buddy_arm-J4_Spindle.dae"/>
+      </geometry>
+    </visual>
+  </link>
   <!--
   =============================================================
@@ -145,3 +159,13 @@
     <origin rpy="${pi} ${pi/2} 0" xyz="-0.004 0.285 0.373"/>
   </joint>
+  <joint name="mcu_base_to_j4_turret_housing_joint" type="fixed">
+    <parent link="mcu_base_link"/>
+    <child link="j4_turret_housing_link"/>
+    <origin rpy="0 ${pi/2} 0" xyz="-0.004 0.285 0.373"/>
+  </joint>
+  <joint name="mcu_base_to_j4_spindle_joint" type="fixed">
+    <parent link="mcu_base_link"/>
+    <child link="j4_spindle_link"/>
+    <origin rpy="${pi/2} ${pi/2} 0" xyz="-0.023 0.347 0.430"/>
+  </joint>
 </robot>

Commit message: Simulation/ros2: add J5 parts in URDF
Signed-off-by: KizEvo <vandungqc03@gmail.com>

File: Simulation/ros2/src/arm_desc/buddyarm_urdf/src/robot_arm.urdf.xacro (robot description, xacro)
@@ -99,4 +99,18 @@
     </visual>
   </link>
+  <link name="j5_arm_link">
+    <visual>
+      <geometry>
+        <mesh filename="package://buddyarm_urdf/mesh/buddy_arm-J5_Arm.dae"/>
+      </geometry>
+    </visual>
+  </link>
+  <link name="j5_spindle_link">
+    <visual>
+      <geometry>
+        <mesh filename="package://buddyarm_urdf/mesh/buddy_arm-J5_Spindle.dae"/>
+      </geometry>
+    </visual>
+  </link>
   <!--
   =============================================================
@@ -169,3 +183,13 @@
     <origin rpy="${pi/2} ${pi/2} 0" xyz="-0.023 0.347 0.430"/>
   </joint>
+  <joint name="mcu_base_to_j5_arm_joint" type="fixed">
+    <parent link="mcu_base_link"/>
+    <child link="j5_arm_link"/>
+    <origin rpy="0 0 0" xyz="-0.040 0.347 0.409"/>
+  </joint>
+  <joint name="mcu_base_to_j5_spindle_joint" type="fixed">
+    <parent link="mcu_base_link"/>
+    <child link="j5_spindle_link"/>
+    <origin rpy="${pi/2} 0 ${pi/2}" xyz="-0.043 0.454 0.430"/>
+  </joint>
 </robot>

Commit message: Simulation/ros2: add J6 part in URDF
Signed-off-by: KizEvo <vandungqc03@gmail.com>

File: Simulation/ros2/src/arm_desc/buddyarm_urdf/src/robot_arm.urdf.xacro (robot description, xacro)
@@ -110,4 +110,11 @@
       <geometry>
         <mesh filename="package://buddyarm_urdf/mesh/buddy_arm-J5_Spindle.dae"/>
+      </geometry>
+    </visual>
+  </link>
+  <link name="j6_arm_link">
+    <visual>
+      <geometry>
+        <mesh filename="package://buddyarm_urdf/mesh/buddy_arm-J6_Arm.dae"/>
       </geometry>
     </visual>
@@ -193,3 +200,8 @@
     <origin rpy="${pi/2} 0 ${pi/2}" xyz="-0.043 0.454 0.430"/>
   </joint>
+  <joint name="mcu_base_to_j6_arm_joint" type="fixed">
+    <parent link="mcu_base_link"/>
+    <child link="j6_arm_link"/>
+    <origin rpy="${pi/2} 0 ${pi/2}" xyz="-0.018 0.454 0.430"/>
+  </joint>
 </robot>

Commit message: Simulation/ros2: fix URDF kinematic tree
Currently every joint  has mcu_base_link as its parent.
This is incorrect, as this means the J2 arm is attached directly to
the base, not to the J1 rotating assembly. When we change the J1 angle
the J2 arm will not follow it.

Simplified tree:

	MCU_Base_Link
		|
	J1 - revolute
		|
	J2 - revolute
		|
	J3 - revolute
		|
		J4 - J5 - J6 - EndEffector

Spindle links are 'fixed' for now, future commit will update to
'revolute'.

Signed-off-by: KizEvo <vandungqc03@gmail.com>

File: Simulation/ros2/src/arm_desc/buddyarm_urdf/src/robot_arm.urdf.xacro (robot description, xacro)
@@ -140,68 +140,75 @@
     <origin xyz="0 0.225 0.025"/>
   </joint>
-  <joint name="mcu_base_to_j1_spindle_joint" type="fixed">
-    <parent link="mcu_base_link"/>
+  <!-- TODO: joint type revolute -->
+  <joint name="j1_base_to_j1_spindle_joint" type="fixed">
+    <parent link="j1_base_link"/>
     <child link="j1_spindle_link"/>
-    <origin xyz="0 0.225 -0.007"/>
-  </joint>
-  <joint name="mcu_base_to_j1_platform_joint" type="fixed">
-    <parent link="mcu_base_link"/>
+    <origin xyz="0 0.150 -0.025"/>
+  </joint>
+  <joint name="j1_spindle_to_j1_platform_joint" type="fixed">
+    <parent link="j1_spindle_link"/>
     <child link="j1_platform_link"/>
-    <origin xyz="0 0.225 0.090"/>
-  </joint>
-  <joint name="mcu_base_to_j2_turret_housing_joint" type="fixed">
-    <parent link="mcu_base_link"/>
+    <origin xyz="0 0 0.097"/>
+  </joint>
+  <joint name="j1_platform_to_j2_turret_housing_joint" type="fixed">
+    <parent link="j1_platform_link"/>
     <child link="j2_turret_housing_link"/>
-    <origin rpy="${pi/2} 0 ${-pi/2}" xyz="-0.021 0.245 0.090"/>
-  </joint>
-  <joint name="mcu_base_to_j2_spindle_joint" type="fixed">
-    <parent link="mcu_base_link"/>
+    <origin rpy="${pi/2} 0 ${-pi/2}" xyz="-0.021 0.020 0"/>
+  </joint>
+  <!-- TODO: joint type revolute -->
+  <joint name="j2_turret_housing_to_j2_spindle_joint" type="fixed">
+    <parent link="j2_turret_housing_link"/>
     <child link="j2_spindle_link"/>
-    <origin rpy="${pi/2} 0 ${pi/2}" xyz="-0.061 0.285 0.140"/>
-  </joint>
-  <joint name="mcu_base_to_j2_tension_ring_joint" type="fixed">
-    <parent link="mcu_base_link"/>
+    <origin rpy="${pi} 0 ${pi}" xyz="-0.040 0.050 0.040"/>
+  </joint>
+  <joint name="j2_spindle_to_j2_tension_ring_joint" type="fixed">
+    <parent link="j2_spindle_link"/>
     <child link="j2_tension_ring_link"/>
-    <origin rpy="${-pi/2} 0 ${pi/2}" xyz="0.010 0.285 0.140"/>
-  </joint>
-  <joint name="mcu_base_to_j2_arm_joint" type="fixed">
-    <parent link="mcu_base_link"/>
+    <origin rpy="${-pi} 0 0" xyz="0 0 0.0710"/>
+  </joint>
+  <joint name="j2_spindle_to_j2_arm_joint" type="fixed">
+    <parent link="j2_spindle_link"/>
     <child link="j2_arm_link"/>
-    <origin rpy="${pi/2} 0 0" xyz="-0.056 0.315 0.110"/>
-  </joint>
-  <joint name="mcu_base_to_j3_bearing_cup_joint" type="fixed">
-    <parent link="mcu_base_link"/>
+    <origin rpy="0 ${-pi/2} -0" xyz="0.0300 -0.0300 0.0050"/>
+  </joint>
+  <joint name="j2_arm_to_j3_bearing_cup_joint" type="fixed">
+    <parent link="j2_arm_link"/>
     <child link="j3_bearing_cup_link"/>
-    <origin rpy="0 ${-pi/2} 0" xyz="-0.024 0.285 0.373"/>
-  </joint>
-  <joint name="mcu_base_to_j3_spindle_joint" type="fixed">
-    <parent link="mcu_base_link"/>
+    <origin rpy="${-pi/2} 0 ${pi/2}" xyz="0.0320 0.2630 0.0300"/>
+  </joint>
+  <!-- TODO: joint type revolute -->
+  <joint name="j3_bearing_cup_to_j3_spindle_joint" type="fixed">
+    <parent link="j3_bearing_cup_link"/>
     <child link="j3_spindle_link"/>
-    <origin rpy="${pi} ${pi/2} 0" xyz="-0.004 0.285 0.373"/>
-  </joint>
-  <joint name="mcu_base_to_j4_turret_housing_joint" type="fixed">
-    <parent link="mcu_base_link"/>
+    <origin rpy="0 0 ${pi}" xyz="0 0 -0.0200"/>
+  </joint>
+  <joint name="j3_spindle_to_j4_turret_housing_joint" type="fixed">
+    <parent link="j3_spindle_link"/>
     <child link="j4_turret_housing_link"/>
-    <origin rpy="0 ${pi/2} 0" xyz="-0.004 0.285 0.373"/>
-  </joint>
-  <joint name="mcu_base_to_j4_spindle_joint" type="fixed">
-    <parent link="mcu_base_link"/>
+    <origin rpy="${-pi} 0 0" xyz="0 0 0"/>
+  </joint>
+  <!-- TODO: joint type revolute -->
+  <joint name="j4_turret_housing_to_j4_spindle_joint" type="fixed">
+    <parent link="j4_turret_housing_link"/>
     <child link="j4_spindle_link"/>
-    <origin rpy="${pi/2} ${pi/2} 0" xyz="-0.023 0.347 0.430"/>
-  </joint>
-  <joint name="mcu_base_to_j5_arm_joint" type="fixed">
-    <parent link="mcu_base_link"/>
+    <origin rpy="${pi/2} 0 0" xyz="-0.0570 0.0620 -0.0190"/>
+  </joint>
+  <joint name="j4_spindle_to_j5_arm_joint" type="fixed">
+    <parent link="j4_spindle_link"/>
     <child link="j5_arm_link"/>
-    <origin rpy="0 0 0" xyz="-0.040 0.347 0.409"/>
-  </joint>
-  <joint name="mcu_base_to_j5_spindle_joint" type="fixed">
-    <parent link="mcu_base_link"/>
+    <origin rpy="${-pi/2} 0 ${pi/2}" xyz="0.0210 -0.0170 0"/>
+  </joint>
+  <!-- TODO: joint type revolute -->
+  <joint name="j5_arm_to_j5_spindle_joint" type="fixed">
+    <parent link="j5_arm_link"/>
     <child link="j5_spindle_link"/>
-    <origin rpy="${pi/2} 0 ${pi/2}" xyz="-0.043 0.454 0.430"/>
-  </joint>
-  <joint name="mcu_base_to_j6_arm_joint" type="fixed">
-    <parent link="mcu_base_link"/>
+    <origin rpy="${pi/2} 0 ${pi/2}" xyz="0.0030 0.1075 0.0210"/>
+  </joint>
+  <joint name="j5_spindle_to_j6_arm_joint" type="fixed">
+    <parent link="j5_spindle_link"/>
     <child link="j6_arm_link"/>
-    <origin rpy="${pi/2} 0 ${pi/2}" xyz="-0.018 0.454 0.430"/>
-  </joint>
+    <origin rpy="0 0 0" xyz="0 0 0.0250"/>
+  </joint>
+  <!-- TODO: joint type revolute -->
+  <!-- TODO: end-effector -->
 </robot>

Commit message: Simulation/ros2: update spindle joints to revolute type
Add axis and limit element for spindle joints.
Update joint type to revolute.
For now, the velocity and effort tag act as placeholder, as these
two tags are required for revolute joint. We're likely to update
this when experimenting with physics.

Signed-off-by: KizEvo <vandungqc03@gmail.com>

File: Simulation/ros2/src/arm_desc/buddyarm_urdf/src/robot_arm.urdf.xacro (robot description, xacro)
@@ -140,9 +140,10 @@
     <origin xyz="0 0.225 0.025"/>
   </joint>
-  <!-- TODO: joint type revolute -->
-  <joint name="j1_base_to_j1_spindle_joint" type="fixed">
+  <joint name="j1_base_to_j1_spindle_joint" type="revolute">
     <parent link="j1_base_link"/>
     <child link="j1_spindle_link"/>
     <origin xyz="0 0.150 -0.025"/>
+    <axis xyz="0 0 1"/>
+    <limit lower="${pi/2}" upper="${-pi/2}" effort="1000.0" velocity="0.2"/>
   </joint>
   <joint name="j1_spindle_to_j1_platform_joint" type="fixed">
@@ -156,9 +157,10 @@
     <origin rpy="${pi/2} 0 ${-pi/2}" xyz="-0.021 0.020 0"/>
   </joint>
-  <!-- TODO: joint type revolute -->
-  <joint name="j2_turret_housing_to_j2_spindle_joint" type="fixed">
+  <joint name="j2_turret_housing_to_j2_spindle_joint" type="revolute">
     <parent link="j2_turret_housing_link"/>
     <child link="j2_spindle_link"/>
     <origin rpy="${pi} 0 ${pi}" xyz="-0.040 0.050 0.040"/>
+    <axis xyz="0 0 1"/>
+    <limit lower="${pi/5}" upper="${-pi/2}" effort="1000.0" velocity="0.2"/>
   </joint>
   <joint name="j2_spindle_to_j2_tension_ring_joint" type="fixed">
@@ -177,9 +179,10 @@
     <origin rpy="${-pi/2} 0 ${pi/2}" xyz="0.0320 0.2630 0.0300"/>
   </joint>
-  <!-- TODO: joint type revolute -->
-  <joint name="j3_bearing_cup_to_j3_spindle_joint" type="fixed">
+  <joint name="j3_bearing_cup_to_j3_spindle_joint" type="revolute">
     <parent link="j3_bearing_cup_link"/>
     <child link="j3_spindle_link"/>
     <origin rpy="0 0 ${pi}" xyz="0 0 -0.0200"/>
+    <axis xyz="0 0 1"/>
+    <limit lower="${pi/2}" upper="${-pi/2}" effort="1000.0" velocity="0.2"/>
   </joint>
   <joint name="j3_spindle_to_j4_turret_housing_joint" type="fixed">
@@ -188,9 +191,10 @@
     <origin rpy="${-pi} 0 0" xyz="0 0 0"/>
   </joint>
-  <!-- TODO: joint type revolute -->
-  <joint name="j4_turret_housing_to_j4_spindle_joint" type="fixed">
+  <joint name="j4_turret_housing_to_j4_spindle_joint" type="revolute">
     <parent link="j4_turret_housing_link"/>
     <child link="j4_spindle_link"/>
     <origin rpy="${pi/2} 0 0" xyz="-0.0570 0.0620 -0.0190"/>
+    <axis xyz="0 0 1"/>
+    <limit lower="${pi * 1.5}" upper="${-pi * 1.5}" effort="1000.0" velocity="0.2"/>
   </joint>
   <joint name="j4_spindle_to_j5_arm_joint" type="fixed">
@@ -199,9 +203,10 @@
     <origin rpy="${-pi/2} 0 ${pi/2}" xyz="0.0210 -0.0170 0"/>
   </joint>
-  <!-- TODO: joint type revolute -->
-  <joint name="j5_arm_to_j5_spindle_joint" type="fixed">
+  <joint name="j5_arm_to_j5_spindle_joint" type="revolute">
     <parent link="j5_arm_link"/>
     <child link="j5_spindle_link"/>
     <origin rpy="${pi/2} 0 ${pi/2}" xyz="0.0030 0.1075 0.0210"/>
+    <axis xyz="0 0 1"/>
+    <limit lower="${pi/2}" upper="${-pi/2}" effort="1000.0" velocity="0.2"/>
   </joint>
   <joint name="j5_spindle_to_j6_arm_joint" type="fixed">
@@ -210,5 +215,5 @@
     <origin rpy="0 0 0" xyz="0 0 0.0250"/>
   </joint>
-  <!-- TODO: joint type revolute -->
+  <!-- TODO: joint type revolute, add this when we have end-effector CAD -->
   <!-- TODO: end-effector -->
 </robot>
