Commit message: Simulation/ros2: add J6 motor and dummy end-effector in URDF
Signed-off-by: KizEvo <vandungqc03@gmail.com>

File: Simulation/ros2/src/buddyarm_urdf/src/robot_arm.urdf.xacro (robot description, xacro)
@@ -117,4 +117,18 @@
       <geometry>
         <mesh filename="package://buddyarm_urdf/mesh/buddy_arm-J6_Arm.dae"/>
+      </geometry>
+    </visual>
+  </link>
+  <link name="j6_motor_link">
+    <visual>
+      <geometry>
+        <mesh filename="package://buddyarm_urdf/mesh/buddy_arm-11HS20-0674D-EGS16-J6-Motor.dae"/>
+      </geometry>
+    </visual>
+  </link>
+  <link name="end_effector">
+    <visual>
+      <geometry>
+        <cylinder length="0.01" radius="0.02"/>
       </geometry>
     </visual>
@@ -215,5 +229,15 @@
     <origin rpy="0 0 0" xyz="0 0 0.0250"/>
   </joint>
-  <!-- TODO: joint type revolute, add this when we have end-effector CAD -->
-  <!-- TODO: end-effector -->
+  <joint name="j6_arm_to_j6_motor_joint" type="fixed">
+    <parent link="j6_arm_link"/>
+    <child link="j6_motor_link"/>
+    <origin rpy="${-pi/2} 0 ${pi/2}" xyz="0.0620 0.0019 0.0262"/>
+  </joint>
+  <joint name="j6_motor_to_end_effector_joint" type="revolute">
+    <parent link="j6_motor_link"/>
+    <child link="end_effector"/>
+    <origin rpy="0.000000 0.000000 ${-pi}" xyz="-0.0019 0.0002 -0.0660"/>
+    <axis xyz="0 0 1"/>
+    <limit lower="${pi/2}" upper="${-pi/2}" effort="1000.0" velocity="0.2"/>
+  </joint>
 </robot>

Commit message: Simulation/ros2: add collision tag to links
Use simple box geometry as collision model.
Help reduce computation time.

End-effectir use cylinder geometry.

Signed-off-by: KizEvo <vandungqc03@gmail.com>

File: Simulation/ros2/src/buddyarm_urdf/src/robot_arm.urdf.xacro (robot description, xacro)
@@ -3,4 +3,18 @@
   <!--
   =============================================================
+                              MACROs
+  =============================================================
+  -->
+  <!-- Params: box: depth/width/heigh and origin xyz -->
+  <xacro:macro name="collision_ele" params="d w h x y z roll pitch yaw">
+    <collision>
+      <geometry>
+        <box size="${d} ${w} ${h}"/>
+      </geometry>
+      <origin rpy="${roll} ${pitch} ${yaw}" xyz="${x} ${y} ${z}"/>
+    </collision>
+  </xacro:macro>
+  <!--
+  =============================================================
                               LINKS
   Origin values based on FreeCAD assembly translation and
@@ -14,4 +28,5 @@
       </geometry>
     </visual>
+    <xacro:collision_ele d="0.150" w="0.370" h="0.018" x="0" y="0.110" z="0.009" roll="0" pitch="0" yaw="0"/>
   </link>
   <link name="j1_base_link">
@@ -28,4 +43,5 @@
       </geometry>
     </visual>
+    <xacro:collision_ele d="0.089" w="0.089" h="0.064" x="0" y="0" z="0.032" roll="0" pitch="0" yaw="0"/>
   </link>
   <link name="j1_platform_link">
@@ -49,4 +65,5 @@
       </geometry>
     </visual>
+    <xacro:collision_ele d="0.076" w="0.203" h="0.060" x="0.0382" y="0.1452" z="0.0300" roll="0" pitch="0" yaw="0"/>
   </link>
   <link name="j2_spindle_link">
@@ -91,4 +108,5 @@
       </geometry>
     </visual>
+    <xacro:collision_ele d="0.060" w="0.042" h="0.044" x="-0.0570" y="0.0320" z="-0.0100" roll="0" pitch="${pi/2}" yaw="${pi/2}"/>
   </link>
   <link name="j4_spindle_link">
@@ -105,4 +123,5 @@
       </geometry>
     </visual>
+    <xacro:collision_ele d="0.125" w="0.042" h="0.020" x="0.002" y="0.0624" z="0.021" roll="${-pi/2}" pitch="0" yaw="${-pi/2}"/>
   </link>
   <link name="j5_spindle_link">
@@ -119,4 +138,5 @@
       </geometry>
     </visual>
+    <xacro:collision_ele d="0.042" w="0.030" h="0.126" x="0.0450" y="0" z="0.0210" roll="0" pitch="${-pi/2}" yaw="${-pi}"/>
   </link>
   <link name="j6_motor_link">
@@ -132,5 +152,13 @@
         <cylinder length="0.01" radius="0.02"/>
       </geometry>
-    </visual>
+      <material name="Cyan">
+        <color rgba="0 1.0 1.0 1.0"/>
+      </material>
+    </visual>
+    <collision>
+      <geometry>
+        <cylinder length="0.01" radius="0.02"/>
+      </geometry>
+    </collision>
   </link>
   <!--

Commit message: Simulation/ros2: refactor robot URDF file
Move joint parts that make up a link into a single
<link> element. <link> element support multiple <visual> element.
Remove redundant links, cleanup <joint> description and <collision>.
We only have 6 joints now.

Signed-off-by: KizEvo <vandungqc03@gmail.com>

File: Simulation/ros2/src/buddyarm_urdf/src/robot_arm.urdf.xacro (robot description, xacro)
@@ -28,70 +28,63 @@
       </geometry>
     </visual>
+    <visual>
+      <geometry>
+        <mesh filename="package://buddyarm_urdf/mesh/buddy_arm-J1_Base.dae"/>
+      </geometry>
+      <origin xyz="0 0.075 0.018"/>
+    </visual>
+    <visual>
+      <geometry>
+        <mesh filename="package://buddyarm_urdf/mesh/buddy_arm-J1_Turret_Housing.dae"/>
+      </geometry>
+      <origin xyz="0 0.225 0.025"/>
+    </visual>
     <xacro:collision_ele d="0.150" w="0.370" h="0.018" x="0" y="0.110" z="0.009" roll="0" pitch="0" yaw="0"/>
   </link>
-  <link name="j1_base_link">
-    <visual>
-      <geometry>
-        <mesh filename="package://buddyarm_urdf/mesh/buddy_arm-J1_Base.dae"/>
-      </geometry>
-    </visual>
-  </link>
-  <link name="j1_turret_housing_link">
-    <visual>
-      <geometry>
-        <mesh filename="package://buddyarm_urdf/mesh/buddy_arm-J1_Turret_Housing.dae"/>
-      </geometry>
-    </visual>
-    <xacro:collision_ele d="0.089" w="0.089" h="0.064" x="0" y="0" z="0.032" roll="0" pitch="0" yaw="0"/>
-  </link>
-  <link name="j1_platform_link">
+  <link name="j1_spindle_link">
+    <visual>
+      <geometry>
+        <mesh filename="package://buddyarm_urdf/mesh/buddy_arm-J1_Spindle.dae"/>
+      </geometry>
+    </visual>
     <visual>
       <geometry>
         <mesh filename="package://buddyarm_urdf/mesh/buddy_arm-J1_Platform.dae"/>
       </geometry>
-    </visual>
-  </link>
-  <link name="j1_spindle_link">
-    <visual>
-      <geometry>
-        <mesh filename="package://buddyarm_urdf/mesh/buddy_arm-J1_Spindle.dae"/>
-      </geometry>
-    </visual>
-  </link>
-  <link name="j2_arm_link">
+      <origin xyz="0 0 0.097"/>
+    </visual>
+    <visual>
+      <geometry>
+        <mesh filename="package://buddyarm_urdf/mesh/buddy_arm-J2_Turret_Housing.dae"/>
+      </geometry>
+      <origin rpy="${pi/2} -0.000000 ${-pi/2}" xyz="-0.0210 0.0200 0.0970"/>
+    </visual>
+    <xacro:collision_ele d="0.089" w="0.089" h="0.064" x="0" y="0" z="0.064" roll="0" pitch="0" yaw="0"/>
+  </link>
+  <link name="j2_spindle_link">
+    <visual>
+      <geometry>
+        <mesh filename="package://buddyarm_urdf/mesh/buddy_arm-J2_Spindle.dae"/>
+      </geometry>
+    </visual>
+    <visual>
+      <geometry>
+        <mesh filename="package://buddyarm_urdf/mesh/buddy_arm-J2_Tension_Ring.dae"/>
+      </geometry>
+      <origin rpy="${-pi} -0.000000 0.000000" xyz="0.0000 -0.0000 0.0710"/>
+    </visual>
     <visual>
       <geometry>
         <mesh filename="package://buddyarm_urdf/mesh/buddy_arm-J2_Arm.dae"/>
       </geometry>
-    </visual>
-    <xacro:collision_ele d="0.076" w="0.203" h="0.060" x="0.0382" y="0.1452" z="0.0300" roll="0" pitch="0" yaw="0"/>
-  </link>
-  <link name="j2_spindle_link">
-    <visual>
-      <geometry>
-        <mesh filename="package://buddyarm_urdf/mesh/buddy_arm-J2_Spindle.dae"/>
-      </geometry>
-    </visual>
-  </link>
-  <link name="j2_tension_ring_link">
-    <visual>
-      <geometry>
-        <mesh filename="package://buddyarm_urdf/mesh/buddy_arm-J2_Tension_Ring.dae"/>
-      </geometry>
-    </visual>
-  </link>
-  <link name="j2_turret_housing_link">
-    <visual>
-      <geometry>
-        <mesh filename="package://buddyarm_urdf/mesh/buddy_arm-J2_Turret_Housing.dae"/>
-      </geometry>
-    </visual>
-  </link>
-  <link name="j3_bearing_cup_link">
+      <origin rpy="0.000000 ${-pi/2} -0.000000" xyz="0.0300 -0.0300 0.0050"/>
+    </visual>
     <visual>
       <geometry>
         <mesh filename="package://buddyarm_urdf/mesh/buddy_arm-J3_Bearing_Cup.dae"/>
       </geometry>
-    </visual>
+      <origin rpy="${-pi} 0.000000 ${pi/2}" xyz="0.0000 0.2330 0.0370"/>
+    </visual>
+    <xacro:collision_ele d="0.076" w="0.163" h="0.060" x="0" y="0.1152" z="0.0432" roll="0" pitch="${-pi/2}" yaw="0"/>
   </link>
   <link name="j3_spindle_link">
@@ -101,12 +94,11 @@
       </geometry>
     </visual>
-  </link>
-  <link name="j4_turret_housing_link">
     <visual>
       <geometry>
         <mesh filename="package://buddyarm_urdf/mesh/buddy_arm-J4_Turret_Housing.dae"/>
       </geometry>
-    </visual>
-    <xacro:collision_ele d="0.060" w="0.042" h="0.044" x="-0.0570" y="0.0320" z="-0.0100" roll="0" pitch="${pi/2}" yaw="${pi/2}"/>
+      <origin rpy="${-pi} 0 0" xyz="0 0 0"/>
+    </visual>
+    <xacro:collision_ele d="0.060" w="0.042" h="0.044" x="-0.0570" y="-0.0320" z="0.0100" roll="0" pitch="${-pi/2}" yaw="${pi/2}"/>
   </link>
   <link name="j4_spindle_link">
@@ -116,12 +108,11 @@
       </geometry>
     </visual>
-  </link>
-  <link name="j5_arm_link">
     <visual>
       <geometry>
         <mesh filename="package://buddyarm_urdf/mesh/buddy_arm-J5_Arm.dae"/>
       </geometry>
-    </visual>
-    <xacro:collision_ele d="0.125" w="0.042" h="0.020" x="0.002" y="0.0624" z="0.021" roll="${-pi/2}" pitch="0" yaw="${-pi/2}"/>
+      <origin rpy="${-pi/2} -0.000000 ${pi/2}" xyz="0.0210 -0.0170 -0.0000"/>
+    </visual>
+    <xacro:collision_ele d="0.125" w="0.042" h="0.020" x="0" y="-0.0150" z="-0.0624" roll="0" pitch="${-pi/2}" yaw="${-pi/2}"/>
   </link>
   <link name="j5_spindle_link">
@@ -131,19 +122,17 @@
       </geometry>
     </visual>
-  </link>
-  <link name="j6_arm_link">
     <visual>
       <geometry>
         <mesh filename="package://buddyarm_urdf/mesh/buddy_arm-J6_Arm.dae"/>
       </geometry>
-    </visual>
-    <xacro:collision_ele d="0.042" w="0.030" h="0.126" x="0.0450" y="0" z="0.0210" roll="0" pitch="${-pi/2}" yaw="${-pi}"/>
-  </link>
-  <link name="j6_motor_link">
+      <origin rpy="0.000000 -0.000000 0.000000" xyz="0.0000 -0.0000 0.0250"/>
+    </visual>
     <visual>
       <geometry>
         <mesh filename="package://buddyarm_urdf/mesh/buddy_arm-11HS20-0674D-EGS16-J6-Motor.dae"/>
       </geometry>
-    </visual>
+      <origin rpy="${-pi/2} -0.000000 ${pi/2}" xyz="0.0620 0.0019 0.0512"/>
+    </visual>
+    <xacro:collision_ele d="0.042" w="0.030" h="0.126" x="0.0450" y="0" z="0.0460" roll="0" pitch="${-pi/2}" yaw="${-pi}"/>
   </link>
   <link name="end_effector">
@@ -172,98 +161,43 @@
   =============================================================
    -->
-  <joint name="mcu_base_to_j1_base_joint" type="fixed">
+  <joint name="j1" type="revolute">
     <parent link="mcu_base_link"/>
-    <child link="j1_base_link"/>
-    <origin xyz="0 0.075 0.018"/>
-  </joint>
-  <joint name="mcu_base_to_j1_turret_housing_joint" type="fixed">
-    <parent link="mcu_base_link"/>
-    <child link="j1_turret_housing_link"/>
-    <origin xyz="0 0.225 0.025"/>
-  </joint>
-  <joint name="j1_base_to_j1_spindle_joint" type="revolute">
-    <parent link="j1_base_link"/>
     <child link="j1_spindle_link"/>
-    <origin xyz="0 0.150 -0.025"/>
-    <axis xyz="0 0 1"/>
-    <limit lower="${pi/2}" upper="${-pi/2}" effort="1000.0" velocity="0.2"/>
-  </joint>
-  <joint name="j1_spindle_to_j1_platform_joint" type="fixed">
+    <origin rpy="0.000000 -0.000000 0.000000" xyz="0.0000 0.2250 -0.0070"/>
+    <axis xyz="0 0 1"/>
+    <limit lower="${pi/2}" upper="${-pi/2}" effort="1000.0" velocity="0.2"/>
+  </joint>
+  <joint name="j2" type="revolute">
     <parent link="j1_spindle_link"/>
-    <child link="j1_platform_link"/>
-    <origin xyz="0 0 0.097"/>
-  </joint>
-  <joint name="j1_platform_to_j2_turret_housing_joint" type="fixed">
-    <parent link="j1_platform_link"/>
-    <child link="j2_turret_housing_link"/>
-    <origin rpy="${pi/2} 0 ${-pi/2}" xyz="-0.021 0.020 0"/>
-  </joint>
-  <joint name="j2_turret_housing_to_j2_spindle_joint" type="revolute">
-    <parent link="j2_turret_housing_link"/>
     <child link="j2_spindle_link"/>
-    <origin rpy="${pi} 0 ${pi}" xyz="-0.040 0.050 0.040"/>
-    <axis xyz="0 0 1"/>
-    <limit lower="${pi/5}" upper="${-pi/2}" effort="1000.0" velocity="0.2"/>
-  </joint>
-  <joint name="j2_spindle_to_j2_tension_ring_joint" type="fixed">
+    <origin rpy="${pi/2} -0.000000 ${pi/2}" xyz="-0.0610 0.0600 0.1470"/>
+    <axis xyz="0 0 1"/>
+    <limit lower="${pi/7}" upper="${-pi/2}" effort="1000.0" velocity="0.2"/>
+  </joint>
+  <joint name="j3" type="revolute">
     <parent link="j2_spindle_link"/>
-    <child link="j2_tension_ring_link"/>
-    <origin rpy="${-pi} 0 0" xyz="0 0 0.0710"/>
-  </joint>
-  <joint name="j2_spindle_to_j2_arm_joint" type="fixed">
-    <parent link="j2_spindle_link"/>
-    <child link="j2_arm_link"/>
-    <origin rpy="0 ${-pi/2} -0" xyz="0.0300 -0.0300 0.0050"/>
-  </joint>
-  <joint name="j2_arm_to_j3_bearing_cup_joint" type="fixed">
-    <parent link="j2_arm_link"/>
-    <child link="j3_bearing_cup_link"/>
-    <origin rpy="${-pi/2} 0 ${pi/2}" xyz="0.0320 0.2630 0.0300"/>
-  </joint>
-  <joint name="j3_bearing_cup_to_j3_spindle_joint" type="revolute">
-    <parent link="j3_bearing_cup_link"/>
     <child link="j3_spindle_link"/>
-    <origin rpy="0 0 ${pi}" xyz="0 0 -0.0200"/>
-    <axis xyz="0 0 1"/>
-    <limit lower="${pi/2}" upper="${-pi/2}" effort="1000.0" velocity="0.2"/>
-  </joint>
-  <joint name="j3_spindle_to_j4_turret_housing_joint" type="fixed">
+    <origin rpy="${pi} -0.000000 ${-pi/2}" xyz="0.0000 0.2330 0.0570"/>
+    <axis xyz="0 0 1"/>
+    <limit lower="${pi/2}" upper="${-pi/2}" effort="1000.0" velocity="0.2"/>
+  </joint>
+  <joint name="j4" type="revolute">
     <parent link="j3_spindle_link"/>
-    <child link="j4_turret_housing_link"/>
-    <origin rpy="${-pi} 0 0" xyz="0 0 0"/>
-  </joint>
-  <joint name="j4_turret_housing_to_j4_spindle_joint" type="revolute">
-    <parent link="j4_turret_housing_link"/>
     <child link="j4_spindle_link"/>
-    <origin rpy="${pi/2} 0 0" xyz="-0.0570 0.0620 -0.0190"/>
+    <origin rpy="${-pi/2} -0.000000 0.000000" xyz="-0.0570 -0.0620 0.0190"/>
     <axis xyz="0 0 1"/>
     <limit lower="${pi * 1.5}" upper="${-pi * 1.5}" effort="1000.0" velocity="0.2"/>
   </joint>
-  <joint name="j4_spindle_to_j5_arm_joint" type="fixed">
+  <joint name="j5" type="revolute">
     <parent link="j4_spindle_link"/>
-    <child link="j5_arm_link"/>
-    <origin rpy="${-pi/2} 0 ${pi/2}" xyz="0.0210 -0.0170 0"/>
-  </joint>
-  <joint name="j5_arm_to_j5_spindle_joint" type="revolute">
-    <parent link="j5_arm_link"/>
     <child link="j5_spindle_link"/>
-    <origin rpy="${pi/2} 0 ${pi/2}" xyz="0.0030 0.1075 0.0210"/>
-    <axis xyz="0 0 1"/>
-    <limit lower="${pi/2}" upper="${-pi/2}" effort="1000.0" velocity="0.2"/>
-  </joint>
-  <joint name="j5_spindle_to_j6_arm_joint" type="fixed">
+    <origin rpy="0.000000 ${pi/2} ${pi/2}" xyz="-0.0000 -0.0200 -0.1075"/>
+    <axis xyz="0 0 1"/>
+    <limit lower="${pi/2}" upper="${-pi/2}" effort="1000.0" velocity="0.2"/>
+  </joint>
+  <joint name="j6" type="revolute">
     <parent link="j5_spindle_link"/>
-    <child link="j6_arm_link"/>
-    <origin rpy="0 0 0" xyz="0 0 0.0250"/>
-  </joint>
-  <joint name="j6_arm_to_j6_motor_joint" type="fixed">
-    <parent link="j6_arm_link"/>
-    <child link="j6_motor_link"/>
-    <origin rpy="${-pi/2} 0 ${pi/2}" xyz="0.0620 0.0019 0.0262"/>
-  </joint>
-  <joint name="j6_motor_to_end_effector_joint" type="revolute">
-    <parent link="j6_motor_link"/>
     <child link="end_effector"/>
-    <origin rpy="0.000000 0.000000 ${-pi}" xyz="-0.0019 0.0002 -0.0660"/>
+    <origin rpy="${pi/2} -0.000000 ${-pi/2}" xyz="0.1280 -0.0000 0.0510"/>
     <axis xyz="0 0 1"/>
     <limit lower="${pi/2}" upper="${-pi/2}" effort="1000.0" velocity="0.2"/>

Commit message: Simulation/ros2: fix limit element lower and upper value
Negative value should be lower and positive value should be higher.

Signed-off-by: KizEvo <vandungqc03@gmail.com>

File: Simulation/ros2/src/buddyarm_urdf/src/robot_arm.urdf.xacro (robot description, xacro)
@@ -166,5 +166,5 @@
     <origin rpy="0.000000 -0.000000 0.000000" xyz="0.0000 0.2250 -0.0070"/>
     <axis xyz="0 0 1"/>
-    <limit lower="${pi/2}" upper="${-pi/2}" effort="1000.0" velocity="0.2"/>
+    <limit lower="${-pi/2}" upper="${pi/2}" effort="1000.0" velocity="1.0"/>
   </joint>
   <joint name="j2" type="revolute">
@@ -173,5 +173,5 @@
     <origin rpy="${pi/2} -0.000000 ${pi/2}" xyz="-0.0610 0.0600 0.1470"/>
     <axis xyz="0 0 1"/>
-    <limit lower="${pi/7}" upper="${-pi/2}" effort="1000.0" velocity="0.2"/>
+    <limit lower="${-pi/7}" upper="${pi/2}" effort="1000.0" velocity="1.0"/>
   </joint>
   <joint name="j3" type="revolute">
@@ -180,5 +180,5 @@
     <origin rpy="${pi} -0.000000 ${-pi/2}" xyz="0.0000 0.2330 0.0570"/>
     <axis xyz="0 0 1"/>
-    <limit lower="${pi/2}" upper="${-pi/2}" effort="1000.0" velocity="0.2"/>
+    <limit lower="${-pi/2}" upper="${pi/2}" effort="1000.0" velocity="1.0"/>
   </joint>
   <joint name="j4" type="revolute">
@@ -187,5 +187,5 @@
     <origin rpy="${-pi/2} -0.000000 0.000000" xyz="-0.0570 -0.0620 0.0190"/>
     <axis xyz="0 0 1"/>
-    <limit lower="${pi * 1.5}" upper="${-pi * 1.5}" effort="1000.0" velocity="0.2"/>
+    <limit lower="${-pi * 1.5}" upper="${pi * 1.5}" effort="1000.0" velocity="1.0"/>
   </joint>
   <joint name="j5" type="revolute">
@@ -194,5 +194,5 @@
     <origin rpy="0.000000 ${pi/2} ${pi/2}" xyz="-0.0000 -0.0200 -0.1075"/>
     <axis xyz="0 0 1"/>
-    <limit lower="${pi/2}" upper="${-pi/2}" effort="1000.0" velocity="0.2"/>
+    <limit lower="${-pi/2}" upper="${pi/2}" effort="1000.0" velocity="1.0"/>
   </joint>
   <joint name="j6" type="revolute">
@@ -201,5 +201,5 @@
     <origin rpy="${pi/2} -0.000000 ${-pi/2}" xyz="0.1280 -0.0000 0.0510"/>
     <axis xyz="0 0 1"/>
-    <limit lower="${pi/2}" upper="${-pi/2}" effort="1000.0" velocity="0.2"/>
+    <limit lower="${-pi/2}" upper="${pi/2}" effort="1000.0" velocity="1.0"/>
   </joint>
 </robot>
